File: KiCad/V2/GameboyCartridgeV2/GameboyCartridgeV2.kicad_sch (KiCad schematic)
At the start: 0 parts

Commit message: Version 2.2
Other:
- title: (none) -> Croco Cartridge
Changed lines of the file:
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@@
 (kicad_sch
-	(version 20250114)
+	(version 20260306)
 	(generator "eeschema")
-	(generator_version "9.0")
+	(generator_version "10.0")
 	(paper "A3")
+	(title_block
+		(title "Croco Cartridge")
+		(date "10/2026")
+		(rev "${VERSION}")
+	)
 	(sheet
 		(at 54.61 57.15)
@@
 		)
 		(fill
-			(color 0 0 0 0.0000)
+			(color 0 0 0 0)
 		)
 		(property "Sheetname" "CPU"
 			(at 54.61 56.4384 0)
+			(show_name no)
+			(do_not_autoplace no)
 			(effects
 				(font
@@
 		(property "Sheetfile" "cpu.kicad_sch"
 			(at 54.61 99.6446 0)
+			(show_name no)
+			(do_not_autoplace no)
 			(effects
 				(font
@@
 		)
 		(instances
-			(project "GameboyCartridgeV2.1"
+			(project "GameboyCartridgeV2"
 				(path "/ec16e1da-c950-4911-941a-a1ab0200cc01"
 					(page "2")
@@
 		)
 		(fill
-			(color 0 0 0 0.0000)
+			(color 0 0 0 0)
 		)
 		(property "Sheetname" "Power_GBBus"
 			(at 167.64 57.7084 0)
+			(show_name no)
+			(do_not_autoplace no)
 			(effects
 				(font
@@
 		(property "Sheetfile" "power.kicad_sch"
 			(at 167.64 105.9946 0)
+			(show_name no)
+			(do_not_autoplace no)
 			(effects
 				(font
@@
 		)
 		(instances
-			(project "GameboyCartridgeV2.1"
+			(project "GameboyCartridgeV2"
 				(path "/ec16e1da-c950-4911-941a-a1ab0200cc01"
 					(page "3")
