File: KiCad/V2/GameboyCartridgeV2/cpu.kicad_sch (KiCad schematic)
At the start: 61 parts, among them J1 USB_C_Receptacle_USB2.0, J2 Micro_SD_Card_Det2, J3 DBG_UART, J4 Conn_01x06, SW1 SW_Push, SW2 SW_Push, U1 USBLC6-2P6, U2 W25Q16JVSSIQ, U3 RP2350_80QFN, U4 W956A8MBYA5I, U5 MCP79510, Y1 12MHz, Y2 32.768kHz

Commit message: Version 2.2
Parts:
- J1: symbol Connector:USB_C_Receptacle_USB2.0 -> Connector:USB_C_Receptacle_USB2.0_16P
- JP1: symbol Jumper:SolderJumper_2_Open -> CrocoV2:SolderJumper_2_Open
- U1: symbol Power_Protection:USBLC6-2P6 -> CrocoV2:USBLC6-2P6
- U2: footprint Package_SO:SOIC-8_5.23x5.23mm_P1.27mm -> Package_SO:SOIC-8_5.3x5.3mm_P1.27mm; symbol Memory_Flash:W25Q128JVS -> CrocoV2:W25Q128JVS
- U3: symbol MCU_RaspberryPi_RP2350:RP2350_80QFN -> CrocoV2:RP2350_80QFN
- U4: symbol local:PSRAM_32M -> CrocoV2:PSRAM_32M
- Y1: symbol Device:Crystal_GND24_Small -> CrocoV2:Crystal_GND24_Small
Connections:
- net GND: now also J1.SH (SHIELD), J2.SH (SHIELD); no longer J1.S1 (SHIELD), J2.11 (SHIELD)
- no-connect marks 8 -> 10
Other:
- title: (none) -> Croco Cartridge
