File: KiCad/V2/GameboyCartridgeV2/power.kicad_sch (KiCad schematic)
At the start: 17 parts, among them J5 CartBus, Q1 CJ2302, U6 AP2112K-3.3, U7 TXB0108PW

Commit message: Version 2.2
Parts:
- J5: symbol Gameboy:CartBus -> CrocoV2:CartBus
- Q1: symbol Device:Q_NMOS_GSD -> Transistor_FET:Q_NMOS_GSD
Connections:
- no-connect marks 0 -> 2
Other:
- title: (none) -> Croco Cartridge
